File: lboard2.kicad_pcb (KiCad board)
At the start: 4 copper layers, 203.2 x 101.6 mm, 225 parts, among them J2 Conn_01x04, J3 PSU_SYNC, J4 PSU_REF, U1 CDCE913PW, U10 AS7C34098A, U11 M25P16-VME, U12 FT232RL, U13 TLV320AIC3204, U14 AMS1117-1.8, U2 STM32F401RBTx, U3 M25P16-VME, U4 USBLC6-2SC6, U5 NCP1117-3.3_SOT223, U6 AMS1117-ADJ, U7 AMS1117-33, U8 L5973D, U9 XC6SLX9-TQG144, Y1 27MHz, Y2 8MHz, Y3 DNP, Y4 ABS25-32.768KHZ-6-T, Y5 DNP32

Commit message: fixed 3v3 supply on CDCE913 output pin ver. bump
Connections:
- C3 pad 1: Net-(C3-Pad1) -> +3V3
- C4 pad 1: Net-(C3-Pad1) -> +3V3
- U1 pad 6: Net-(C3-Pad1) -> +3V3
- U1 pad 7: Net-(C3-Pad1) -> +3V3
Routing:
- net +3V3: track 1205.9 -> 1241.6 mm, vias 60 -> 61
- net Net-(C3-Pad1): track 20.6 -> 0.00 mm
Other:
- board text added: "lboard v2.8.000 2018-09-27"
- board text removed: "lboard v2.2.002 2018-08-27"

Commit message: schematics pdf and board updates
Routing:
- net /CODEC/LOL: track 112.4 -> 120.4 mm
- net /CODEC/LOR: track 102.9 -> 110.6 mm
Changed lines of the file:
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@@
   (general
     (links 622)
-    (no_connects 3)
+    (no_connects 2)
     (area 50.749999 50.749999 254.050001 152.450001)
     (thickness 1.6)
@@
       (drillshape 0)
       (scaleselection 1)
-      (outputdirectory plot/gerber-v2.1/lboard-gerber-v2.2.002/))
+      (outputdirectory plot/gerber-v2.8/lboard-gerber-v2.8.000/))
   )
   (net 0 "")
@@
   (segment (start 98.933 89.662) (end 99.060705 89.534295) (width 0.25) (layer F.Cu) (net 6))
   (segment (start 99.060705 89.534295) (end 99.060705 89.40359) (width 0.25) (layer F.Cu) (net 6))
-  (via (at 99.060705 89.40359) (size 0.6) (drill 0.4) (layers F.Cu B.Cu) (net 6) (status 1000000))
+  (via (at 99.060705 89.40359) (size 0.6) (drill 0.4) (layers F.Cu B.Cu) (net 6))
   (segment (start 98.933 94.488) (end 98.933 89.662) (width 0.25) (layer F.Cu) (net 6))
   (segment (start 101.473 97.028) (end 98.933 94.488) (width 0.25) (layer F.Cu) (net 6))
@@
   (segment (start 118.257 73.152) (end 116.713 73.152) (width 0.25) (layer F.Cu) (net 35))
   (via (at 116.713 73.152) (size 0.6) (drill 0.4) (layers F.Cu B.Cu) (net 35))
+  (segment (start 74.295 77.978) (end 75.578 77.978) (width 0.25) (layer F.Cu) (net 36))
+  (segment (start 142.748 71.884) (end 135.128001 64.264001) (width 0.25) (layer F.Cu) (net 36))
+  (segment (start 71.627999 57.02159) (end 71.627999 75.311) (width 0.25) (layer F.Cu) (net 36))
+  (segment (start 130.359989 51.619989) (end 77.0296 51.619989) (width 0.25) (layer F.Cu) (net 36))
+  (segment (start 135.128001 56.388001) (end 130.359989 51.619989) (width 0.25) (layer F.Cu) (net 36))
+  (segment (start 77.0296 51.619989) (end 71.627999 57.02159) (width 0.25) (layer F.Cu) (net 36))
+  (segment (start 135.128001 64.264001) (end 135.128001 56.388001) (width 0.25) (layer F.Cu) (net 36))
   (segment (start 142.748 72.009) (end 142.748 71.884) (width 0.25) (layer F.Cu) (net 36))
+  (segment (start 71.627999 75.311) (end 74.295 77.978) (width 0.25) (layer F.Cu) (net 36))
   (segment (start 75.578 77.978) (end 75.725 78.125) (width 0.25) (layer F.Cu) (net 36))
-  (segment (start 142.748 71.884) (end 135.128 64.264) (width 0.25) (layer F.Cu) (net 36))
-  (segment (start 74.295 77.978) (end 75.578 77.978) (width 0.25) (layer F.Cu) (net 36))
   (segment (start 75.725 78.125) (end 75.725 78.725) (width 0.25) (layer F.Cu) (net 36))
-  (segment (start 135.128 64.264) (end 135.128 61.595) (width 0.25) (layer F.Cu) (net 36))
-  (segment (start 135.128 61.595) (end 130.048 56.515) (width 0.25) (layer F.Cu) (net 36))
-  (segment (start 130.048 56.515) (end 73.152 56.515) (width 0.25) (layer F.Cu) (net 36))
-  (segment (start 73.152 56.515) (end 71.628 58.039) (width 0.25) (layer F.Cu) (net 36))
-  (segment (start 71.628 58.039) (end 71.628 75.311) (width 0.25) (layer F.Cu) (net 36))
-  (segment (start 71.628 75.311) (end 74.295 77.978) (width 0.25) (layer F.Cu) (net 36))
   (segment (start 142.748 69.509) (end 146.999 69.509) (width 0.25) (layer F.Cu) (net 37))
   (segment (start 146.999 69.509) (end 149.352 67.156) (width 0.25) (layer F.Cu) (net 37))
@@
   (segment (start 127.04 73.279) (end 127.167 73.152) (width 0.25) (layer F.Cu) (net 38))
   (via (at 125.222 73.279) (size 0.6) (drill 0.4) (layers F.Cu B.Cu) (net 38))
+  (segment (start 72.07801 75.1246) (end 72.07801 57.20799) (width 0.25) (layer F.Cu) (net 39))
+  (segment (start 77.216 52.07) (end 130.048 52.07) (width 0.25) (layer F.Cu) (net 39))
+  (segment (start 134.67799 65.898992) (end 141.862999 73.084001) (width 0.25) (layer F.Cu) (net 39))
+  (segment (start 74.29641 77.343) (end 72.07801 75.1246) (width 0.25) (layer F.Cu) (net 39))
+  (segment (start 75.57941 77.343) (end 74.29641 77.343) (width 0.25) (layer F.Cu) (net 39))
   (segment (start 76.225 78.725) (end 76.225 77.98859) (width 0.25) (layer F.Cu) (net 39))
   (segment (start 76.225 77.98859) (end 75.57941 77.343) (width 0.25) (layer F.Cu) (net 39))
-  (segment (start 75.57941 77.343) (end 74.29641 77.343) (width 0.25) (layer F.Cu) (net 39))
-  (segment (start 74.29641 77.343) (end 72.07801 75.1246) (width 0.25) (layer F.Cu) (net 39))
-  (segment (start 72.07801 75.1246) (end 72.07801 58.453988) (width 0.25) (layer F.Cu) (net 39))
-  (segment (start 134.67799 62.169988) (end 134.67799 65.898992) (width 0.25) (layer F.Cu) (net 39))
-  (segment (start 72.07801 58.453988) (end 73.566988 56.96501) (width 0.25) (layer F.Cu) (net 39))
-  (segment (start 73.566988 56.96501) (end 129.473012 56.96501) (width 0.25) (layer F.Cu) (net 39))
-  (segment (start 129.473012 56.96501) (end 134.67799 62.169988) (width 0.25) (layer F.Cu) (net 39))
-  (segment (start 134.67799 65.898992) (end 141.862999 73.084001) (width 0.25) (layer F.Cu) (net 39))
-  (segment (start 141.862999 73.084001) (end 150.175999 73.084001) (width 0.25) (layer F.Cu) (net 39))
-  (segment (start 151.017 72.243) (end 151.892 72.243) (width 0.25) (layer F.Cu) (net 39))
+  (segment (start 72.07801 57.20799) (end 77.216 52.07) (width 0.25) (layer F.Cu) (net 39))
+  (segment (start 130.048 52.07) (end 134.67799 56.69999) (width 0.25) (layer F.Cu) (net 39))
   (segment (start 150.175999 73.084001) (end 151.017 72.243) (width 0.25) (layer F.Cu) (net 39))
+  (segment (start 151.017 72.243) (end 151.892 72.243) (width 0.25) (layer F.Cu) (net 39))
+  (segment (start 134.67799 56.69999) (end 134.67799 65.898992) (width 0.25) (layer F.Cu) (net 39))
+  (segment (start 141.862999 73.084001) (end 150.175999 73.084001) (width 0.25) (layer F.Cu) (net 39))
   (segment (start 159.512 67.056) (end 158.612 67.056) (width 0.25) (layer F.Cu) (net 40))
   (segment (start 152.767 69.743) (end 151.892 69.743) (width 0.25) (layer F.Cu) (net 40))

Commit message: CSI_B must be left unconnected! ver. bump
Parts:
- R13: value 100 -> 390
- R7: value 10k -> DNP
Connections:
- U9 pad 64: GND -> Net-(U9-Pad64)
Routing:
- net GND: track 2972.4 -> 2963.5 mm, vias 132 -> 131
- net Net-(U9-Pad64): track 0.00 -> 7.36 mm
Other:
- board text added: "lboard v2.9.000 2019-03-22"
- board text removed: "lboard v2.8.000 2018-09-27"
Changed lines of the file:
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@@
 (kicad_pcb (version 4) (host pcbnew 4.0.7-e2-6376~58~ubuntu16.04.1)
   (general
-    (links 622)
+    (links 621)
     (no_connects 2)
     (area 50.749999 50.749999 254.050001 152.450001)
     (thickness 1.6)
     (drawings 17)
-    (tracks 4022)
+    (tracks 4019)
     (zones 0)
     (modules 225)
-    (nets 256)
+    (nets 257)
   )
   (page A4)
@@
   (net 254 "Net-(R47-Pad2)")
   (net 255 "Net-(R48-Pad2)")
+  (net 256 "Net-(U9-Pad64)")
   (net_class Default "This is the default net class."
     (clearance 0.2)
@@
     (add_net "Net-(U2-Pad62)")
     (add_net "Net-(U8-Pad9)")
+    (add_net "Net-(U9-Pad64)")
     (add_net "Net-(U9-Pad72)")
     (add_net "Net-(Y4-Pad2)")
@@
       (effects (font (size 1 1) (thickness 0.15)))
     )
-    (fp_text value 10k (at 0 1.75 180) (layer F.Fab)
+    (fp_text value DNP (at 0 1.75 180) (layer F.Fab)
       (effects (font (size 1 1) (thickness 0.15)))
     )
@@
       (net 6 +3V3))
     (pad 64 smd rect (at 4.75 10.7) (size 1.55 0.3) (layers F.Cu F.Paste F.Mask)
-      (net 2 GND))
+      (net 256 "Net-(U9-Pad64)"))
     (pad 65 smd rect (at 5.25 10.7) (size 1.55 0.3) (layers F.Cu F.Paste F.Mask)
       (net 63 /FPGA/CBUS_DATA))
@@
       (effects (font (size 1 1) (thickness 0.15)))
     )
-    (fp_text value 100 (at 4.238 -0.127 180) (layer F.Fab)
+    (fp_text value 390 (at 4.238 -0.127 180) (layer F.Fab)
       (effects (font (size 1 1) (thickness 0.15)))
     )
@@
     (effects (font (size 1.5 1.5) (thickness 0.3)))
   )
-  (gr_text "lboard v2.8.000\n2018-09-27" (at 61.722 71.501) (layer F.SilkS)
+  (gr_text "lboard v2.9.000\n2019-03-22" (at 61.722 71.501) (layer F.SilkS)
     (effects (font (size 1.5 1.5) (thickness 0.3)))
   )
@@
   (segment (start 197.104 101.172) (end 200.192 98.084) (width 0.25) (layer In1.Cu) (net 2))
   (segment (start 212.979 107.188) (end 208.534 107.188) (width 0.25) (layer In1.Cu) (net 2))
-  (segment (start 208.534 107.188) (end 204.978 110.744) (width 0.25) (layer In1.Cu) (net 2))
   (segment (start 174.625 120.396) (end 172.085 120.396) (width 0.25) (layer In1.Cu) (net 2))
   (segment (start 172.085 120.396) (end 169.799 118.11) (width 0.25) (layer In1.Cu) (net 2))
@@
   (segment (start 201.326324 111.156324) (end 203.327 113.157) (width 0.25) (layer In1.Cu) (net 2))
   (segment (start 203.327 113.157) (end 203.327 112.395) (width 0.25) (layer In1.Cu) (net 2))
-  (segment (start 203.327 112.395) (end 204.978 110.744) (width 0.25) (layer In1.Cu) (net 2))
   (segment (start 208.788 112.522) (end 203.962 112.522) (width 0.25) (layer In1.Cu) (net 2))
   (segment (start 203.962 112.522) (end 203.327 113.157) (width 0.25) (layer In1.Cu) (net 2))
@@
   (segment (start 206.426 112.446) (end 204.038 112.446) (width 0.25) (layer F.Cu) (net 2))
   (via (at 203.327 113.157) (size 0.6) (drill 0.4) (layers F.Cu B.Cu) (net 2))
-  (segment (start 206.426 110.446) (end 205.276 110.446) (width 0.25) (layer F.Cu) (net 2))
-  (segment (start 205.276 110.446) (end 204.978 110.744) (width 0.25) (layer F.Cu) (net 2))
-  (via (at 204.978 110.744) (size 0.6) (drill 0.4) (layers F.Cu B.Cu) (net 2))
   (segment (start 208.488001 112.821999) (end 208.788 112.522) (width 0.25) (layer F.Cu) (net 2))
   (segment (start 208.376 112.934) (end 208.488001 112.821999) (width 0.25) (layer F.Cu) (net 2))
@@
   (segment (start 123.536 101.01) (end 123.618 101.092) (width 0.25) (layer F.Cu) (net 255))
   (segment (start 120.29 101.01) (end 119.79 101.01) (width 0.25) (layer F.Cu) (net 255))
+  (segment (start 208.534 107.188) (end 204.978 110.744) (width 0.25) (layer In1.Cu) (net 256))
+  (segment (start 203.327 112.395) (end 204.978 110.744) (width 0.25) (layer In1.Cu) (net 256))
   (zone (net 0) (net_name "") (layer B.Cu) (hatch edge 0.508)
     (connect_pads (clearance 0.508))

Commit message: silkscreen description on a configuration bus
Routing:
- net GND: track 2963.5 -> 2970.8 mm
- net Net-(U9-Pad64): track 7.36 -> 0.00 mm
Other:
- board text added: "busy"
- board text added: "cclk"
- board text added: "din"
- board text added: "done"
- board text added: "gnd"
- board text added: "initb"
- board text added: "lboard v2.9.001 2019-03-22"
- board text added: "progb"
- board text removed: "lboard v2.9.000 2019-03-22"
Changed lines of the file:
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@@
     (links 621)
     (no_connects 2)
-    (area 50.749999 50.749999 254.050001 152.450001)
+    (area 16.835716 30.32 260.024572 157.747001)
     (thickness 1.6)
-    (drawings 17)
+    (drawings 24)
     (tracks 4019)
     (zones 0)
@@
   )
   (page A4)
+  (title_block
+    (rev 2.9.001)
+  )
   (layers
     (0 F.Cu signal)
@@
     )
   )
+  (gr_text gnd (at 142.24 132.715 270) (layer F.SilkS)
+    (effects (font (size 1.5 1.5) (thickness 0.3)))
+  )
+  (gr_text din (at 157.48 132.715 270) (layer F.SilkS)
+    (effects (font (size 1.5 1.5) (thickness 0.3)))
+  )
+  (gr_text done (at 154.94 133.35 270) (layer F.SilkS)
+    (effects (font (size 1.5 1.5) (thickness 0.3)))
+  )
+  (gr_text busy (at 152.4 133.35 270) (layer F.SilkS)
+    (effects (font (size 1.5 1.5) (thickness 0.3)))
+  )
+  (gr_text cclk (at 149.86 133.35 270) (layer F.SilkS)
+    (effects (font (size 1.5 1.5) (thickness 0.3)))
+  )
+  (gr_text initb (at 147.32 133.35 270) (layer F.SilkS)
+    (effects (font (size 1.5 1.5) (thickness 0.3)))
+  )
+  (gr_text progb (at 144.78 133.985 270) (layer F.SilkS)
+    (effects (font (size 1.5 1.5) (thickness 0.3)))
+  )
   (gr_text "LINE OUT" (at 145.288 57.15 90) (layer F.SilkS)
     (effects (font (size 1.5 1.5) (thickness 0.3)))
@@
     (effects (font (size 1.5 1.5) (thickness 0.3)))
   )
-  (gr_text "lboard v2.9.000\n2019-03-22" (at 61.722 71.501) (layer F.SilkS)
+  (gr_text "lboard v2.9.001\n2019-03-22" (at 61.722 71.501) (layer F.SilkS)
     (effects (font (size 1.5 1.5) (thickness 0.3)))
   )
@@
   (via (at 200.192 98.084) (size 0.6) (drill 0.4) (layers F.Cu B.Cu) (net 2))
   (segment (start 200.192 99.568) (end 200.192 98.084) (width 0.25) (layer B.Cu) (net 2))
+  (segment (start 208.534 107.188) (end 204.978 110.744) (width 0.25) (layer In1.Cu) (net 2))
+  (segment (start 203.327 112.395) (end 204.978 110.744) (width 0.25) (layer In1.Cu) (net 2))
   (segment (start 149.395264 104.394) (end 148.971 104.394) (width 0.25) (layer B.Cu) (net 3))
   (segment (start 149.97101 104.394) (end 149.395264 104.394) (width 0.25) (layer B.Cu) (net 3))
@@
   (segment (start 123.536 101.01) (end 123.618 101.092) (width 0.25) (layer F.Cu) (net 255))
   (segment (start 120.29 101.01) (end 119.79 101.01) (width 0.25) (layer F.Cu) (net 255))
-  (segment (start 208.534 107.188) (end 204.978 110.744) (width 0.25) (layer In1.Cu) (net 256))
-  (segment (start 203.327 112.395) (end 204.978 110.744) (width 0.25) (layer In1.Cu) (net 256))
   (zone (net 0) (net_name "") (layer B.Cu) (hatch edge 0.508)
     (connect_pads (clearance 0.508))

Commit message: Schematics updates
 U1 CDCDE913  Vctrl pin resistor is marked as DNP. Schematics pdf, gerbers and the photo were updated.
Other:
- board text added: "lboard v2.9.002 2019-03-23"
- board text removed: "lboard v2.9.001 2019-03-22"
Changed lines of the file:
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@@
     (links 621)
     (no_connects 2)
-    (area 16.835716 30.32 260.024572 157.747001)
+    (area 50.749999 50.749999 254.050001 152.450001)
     (thickness 1.6)
     (drawings 24)
@@
   (page A4)
   (title_block
-    (rev 2.9.001)
+    (rev 2.9.002)
   )
   (layers
@@
       (drillshape 0)
       (scaleselection 1)
-      (outputdirectory plot/gerber-v2.8/lboard-gerber-v2.8.000/))
+      (outputdirectory plot/gerber-v2.9/lboard-gerber-v2.9.002/))
   )
   (net 0 "")
@@
     (effects (font (size 1.5 1.5) (thickness 0.3)))
   )
-  (gr_text "lboard v2.9.001\n2019-03-22" (at 61.722 71.501) (layer F.SilkS)
+  (gr_text "lboard v2.9.002\n2019-03-23" (at 61.722 71.501) (layer F.SilkS)
     (effects (font (size 1.5 1.5) (thickness 0.3)))
   )

Commit message: lboard2	added pullup resistors on a codec i2c bus
Parts:
- added R49: 10k, Resistors_SMD:R_0805_HandSoldering, F.Cu at (100.2, 72.4)
- added R50: 10k, Resistors_SMD:R_0805_HandSoldering, F.Cu at (100.3, 76.2)
- R6: value 10k -> 10k DNP
Routing:
- net +3V3: track 1241.6 -> 1262.7 mm, vias 61 -> 63
- net /CODEC/CODEC_SCL: track 146.7 -> 151.1 mm
- net /CODEC/CODEC_SDA: track 148.5 -> 152.7 mm
Other:
- board text added: "lboard v2.9.005 2019-04-04"
- board text removed: "lboard v2.9.002 2019-03-23"
Changed lines of the file:
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@@
 (kicad_pcb (version 4) (host pcbnew 4.0.7-e2-6376~58~ubuntu16.04.1)
   (general
-    (links 621)
-    (no_connects 2)
+    (links 625)
+    (no_connects 5)
     (area 50.749999 50.749999 254.050001 152.450001)
     (thickness 1.6)
     (drawings 24)
-    (tracks 4019)
+    (tracks 4027)
     (zones 0)
-    (modules 225)
+    (modules 227)
     (nets 257)
   )
@@
       (effects (font (size 1 1) (thickness 0.15)))
     )
-    (fp_text value 10k (at 0 1.75 180) (layer F.Fab)
+    (fp_text value "10k DNP" (at 0 1.75 180) (layer F.Fab)
       (effects (font (size 1 1) (thickness 0.15)))
     )
@@
     )
   )
+  (module Resistors_SMD:R_0805_HandSoldering (layer F.Cu)
+    (at 100.25 72.39 180)
+    (descr "Resistor SMD 0805, hand soldering")
+    (tags "resistor 0805")
+    (attr smd)
+    (fp_text reference R49 (at -3.89 1.27 180) (layer F.SilkS)
+      (effects (font (size 1 1) (thickness 0.15)))
+    )
+    (fp_text value 10k (at 0 1.75 180) (layer F.Fab)
+      (effects (font (size 1 1) (thickness 0.15)))
+    )
+    (fp_text user %R (at 0 0 180) (layer F.Fab)
+      (effects (font (size 0.5 0.5) (thickness 0.075)))
+    )
+    (fp_line (start -1 0.62) (end -1 -0.62) (layer F.Fab) (width 0.1))
+    (fp_line (start 1 0.62) (end -1 0.62) (layer F.Fab) (width 0.1))
+    (fp_line (start 1 -0.62) (end 1 0.62) (layer F.Fab) (width 0.1))
+    (fp_line (start -1 -0.62) (end 1 -0.62) (layer F.Fab) (width 0.1))
+    (fp_line (start 0.6 0.88) (end -0.6 0.88) (layer F.SilkS) (width 0.12))
+    (fp_line (start -0.6 -0.88) (end 0.6 -0.88) (layer F.SilkS) (width 0.12))
+    (fp_line (start -2.35 -0.9) (end 2.35 -0.9) (layer F.CrtYd) (width 0.05))
+    (fp_line (start -2.35 -0.9) (end -2.35 0.9) (layer F.CrtYd) (width 0.05))
+    (fp_line (start 2.35 0.9) (end 2.35 -0.9) (layer F.CrtYd) (width 0.05))
+    (fp_line (start 2.35 0.9) (end -2.35 0.9) (layer F.CrtYd) (width 0.05))
+    (pad 1 smd rect (at -1.35 0 180) (size 1.5 1.3) (layers F.Cu F.Paste F.Mask)
+      (net 6 +3V3))
+    (pad 2 smd rect (at 1.35 0 180) (size 1.5 1.3) (layers F.Cu F.Paste F.Mask)
+      (net 69 /CODEC/CODEC_SDA))
+    (model ${KISYS3DMOD}/Resistors_SMD.3dshapes/R_0805.wrl
+      (at (xyz 0 0 0))
+      (scale (xyz 1 1 1))
+      (rotate (xyz 0 0 0))
+    )
+  )
+  (module Resistors_SMD:R_0805_HandSoldering (layer F.Cu)
+    (at 100.33 76.2 180)
+    (descr "Resistor SMD 0805, hand soldering")
+    (tags "resistor 0805")
+    (attr smd)
+    (fp_text reference R50 (at -4.445 0.635 180) (layer F.SilkS)
+      (effects (font (size 1 1) (thickness 0.15)))
+    )
+    (fp_text value 10k (at 0 1.75 180) (layer F.Fab)
+      (effects (font (size 1 1) (thickness 0.15)))
+    )
+    (fp_text user %R (at 0 0 180) (layer F.Fab)
+      (effects (font (size 0.5 0.5) (thickness 0.075)))
+    )
+    (fp_line (start -1 0.62) (end -1 -0.62) (layer F.Fab) (width 0.1))
+    (fp_line (start 1 0.62) (end -1 0.62) (layer F.Fab) (width 0.1))
+    (fp_line (start 1 -0.62) (end 1 0.62) (layer F.Fab) (width 0.1))
+    (fp_line (start -1 -0.62) (end 1 -0.62) (layer F.Fab) (width 0.1))
+    (fp_line (start 0.6 0.88) (end -0.6 0.88) (layer F.SilkS) (width 0.12))
+    (fp_line (start -0.6 -0.88) (end 0.6 -0.88) (layer F.SilkS) (width 0.12))
+    (fp_line (start -2.35 -0.9) (end 2.35 -0.9) (layer F.CrtYd) (width 0.05))
+    (fp_line (start -2.35 -0.9) (end -2.35 0.9) (layer F.CrtYd) (width 0.05))
+    (fp_line (start 2.35 0.9) (end 2.35 -0.9) (layer F.CrtYd) (width 0.05))
+    (fp_line (start 2.35 0.9) (end -2.35 0.9) (layer F.CrtYd) (width 0.05))
+    (pad 1 smd rect (at -1.35 0 180) (size 1.5 1.3) (layers F.Cu F.Paste F.Mask)
+      (net 6 +3V3))
+    (pad 2 smd rect (at 1.35 0 180) (size 1.5 1.3) (layers F.Cu F.Paste F.Mask)
+      (net 68 /CODEC/CODEC_SCL))
+    (model ${KISYS3DMOD}/Resistors_SMD.3dshapes/R_0805.wrl
+      (at (xyz 0 0 0))
+      (scale (xyz 1 1 1))
+      (rotate (xyz 0 0 0))
+    )
+  )
   (gr_text gnd (at 142.24 132.715 270) (layer F.SilkS)
     (effects (font (size 1.5 1.5) (thickness 0.3)))
@@
     (effects (font (size 1.5 1.5) (thickness 0.3)))
   )
-  (gr_text "lboard v2.9.002\n2019-03-23" (at 61.722 71.501) (layer F.SilkS)
+  (gr_text "lboard v2.9.005\n2019-04-04" (at 61.722 71.501) (layer F.SilkS)
     (effects (font (size 1.5 1.5) (thickness 0.3)))
   )
@@
   (segment (start 147.086 117.856) (end 146.304 117.074) (width 0.25) (layer F.Cu) (net 5))
   (segment (start 146.304 117.074) (end 146.304 115.824) (width 0.25) (layer F.Cu) (net 5))
+  (via (at 102.87 76.2) (size 0.6) (drill 0.4) (layers F.Cu B.Cu) (net 6))
+  (segment (start 101.68 76.2) (end 102.87 76.2) (width 0.25) (layer F.Cu) (net 6))
+  (segment (start 102.87 72.39) (end 102.87 85.594295) (width 0.25) (layer In2.Cu) (net 6))
+  (segment (start 102.87 85.594295) (end 99.060705 89.40359) (width 0.25) (layer In2.Cu) (net 6))
+  (via (at 102.87 72.39) (size 0.6) (drill 0.4) (layers F.Cu B.Cu) (net 6))
+  (segment (start 101.6 72.39) (end 102.87 72.39) (width 0.25) (layer F.Cu) (net 6))
   (segment (start 127.762 89.348999) (end 99.060705 89.40359) (width 1) (layer In2.Cu) (net 6))
   (segment (start 99.060705 89.40359) (end 76.699999 89.348999) (width 1) (layer In2.Cu) (net 6))
@@
   (segment (start 83.439 93.98) (end 82.169 93.98) (width 0.25) (layer B.Cu) (net 67))
   (segment (start 82.169 93.98) (end 82.169 94.742) (width 0.25) (layer B.Cu) (net 67))
+  (segment (start 94.615 76.2) (end 98.98 76.2) (width 0.25) (layer F.Cu) (net 68))
   (segment (start 206.426 111.446) (end 199.099901 111.446) (width 0.25) (layer F.Cu) (net 68))
   (segment (start 197.959637 112.586264) (end 177.776493 112.586264) (width 0.25) (layer F.Cu) (net 68))
@@
   (segment (start 128.651 118.56001) (end 128.46601 118.56001) (width 0.25) (layer F.Cu) (net 68))
   (segment (start 128.651 118.56001) (end 127.93914 118.56001) (width 0.25) (layer F.Cu) (net 68))
+  (segment (start 94.615 72.39) (end 98.9 72.39) (width 0.25) (layer F.Cu) (net 69))
   (segment (start 177.585616 111.758976) (end 143.219609 111.758976) (width 0.25) (layer F.Cu) (net 69))
   (segment (start 129.099987 117.415987) (end 121.330999 109.646999) (width 0.25) (layer F.Cu) (net 69))

Commit message: lboard2 v2.9.006
added debug headers for spi flash, addedd  R51 - serial termination resistor for a CBUS_DATA line
Parts:
- added J_SPIFLASHF_DBG2: Conn_01x05, Pin_Headers:Pin_Header_Straight_1x05_Pitch2.54mm, F.Cu at (234.9, 78.7)
- added J_SPIFLASH_DBG1: Conn_01x05, Pin_Headers:Pin_Header_Straight_1x05_Pitch2.54mm, F.Cu at (176.5, 122.6)
- added R51: 10, Resistors_SMD:R_0805_HandSoldering, F.Cu at (201.9, 121.3)
- moved R7 2.93 mm to (186.1, 120.0)
- moved R26 1.48 mm to (235.5, 74.3)
Connections:
- U9 pad 65: /FPGA/CBUS_DATA -> Net-(R51-Pad1)
Routing:
- net /MCU/TRST: track 133.5 -> 23.0 mm
- net /FPGA/SPIFL_MISO: track 25.8 -> 66.0 mm, vias 0 -> 1
- net /MCU/SPIFL_NSS: track 40.7 -> 58.2 mm
- net /FPGA/CBUS_DATA: track 100.5 -> 85.2 mm
- net Net-(R51-Pad1): track 0.00 -> 12.9 mm
- net /MCU/SPIFL_MOSI: track 26.5 -> 38.0 mm
- net /FPGA/SPIFL_MOSI: track 21.6 -> 31.9 mm, vias 0 -> 1
- net /MCU/SPIFL_SCK: track 26.8 -> 35.9 mm
- net /MCU/SPIFL_MISO: track 43.0 -> 51.7 mm
- net /FPGA/SPIFL_CLK: track 24.1 -> 32.3 mm, vias 0 -> 1
- net +3V3: track 1262.7 -> 1255.9 mm
- net /FPGA/SPIFL_CS: track 37.8 -> 42.7 mm, vias 0 -> 1
- net /FPGA/CBUS_BUSY: track 109.4 -> 110.5 mm
- net /FPGA/CBUS_CLOCK: track 95.9 -> 96.8 mm
- net /FPGA/USB_UART_TX: track 208.0 -> 207.2 mm
Other:
- board text added: "ck"
- board text added: "cs"
- board text added: "lboard v2.9.006 2019-04-06"
- board text added: "miso"
- board text added: "mo"
- board text added: "mosi"
- board text removed: "lboard v2.9.005 2019-04-04"
