File: lboard2.kicad_pcb (KiCad board)
At the start: 4 copper layers, 203.2 x 101.6 mm, 230 parts, among them J2 Conn_01x04, J3 PSU_SYNC, J4 PSU_REF, U1 CDCE913PW, U10 AS7C34098A, U11 M25P16-VME, U12 FT232RL, U13 TLV320AIC3204, U14 AMS1117-1.8, U2 STM32F401RBTx, U3 M25P16-VME, U4 USBLC6-2SC6, U5 NCP1117-3.3_SOT223, U6 AMS1117-ADJ, U7 AMS1117-33, U8 L5973D, U9 XC6SLX9-TQG144, Y1 27MHz, Y2 8MHz, Y3 DNP, Y4 ABS25-32.768KHZ-6-T, Y5 DNP32

Commit message: codec word select and bit clock lines are now routed to an fpga global clock pins
Parts:
- renumbered J_COD_BCLK1 to BCLK, J_COD_CLKAU1 to CLKAUX, J_TSTCLKCODEC1 to CLKCODEC, J_COD_DIN1 to DIN, J_COD_DOUT1 to DOUT, J_COD_RST1 to RST, J_COD_SCL1 to SCL, J_COD_SDA1 to SDA, J_COD_WCLK1 to WCLK
Connections:
- J_X2 pad 13: /FPGA/X2_L31N -> Net-(J_X2-Pad13)
- J_X2 pad 15: /FPGA/X2_L31P -> Net-(J_X2-Pad15)
- U9 pad 50: /FPGA/X2_L31N -> /CODEC/CODEC_BCLK
- U9 pad 51: /FPGA/X2_L31P -> /CODEC/CODEC_WCLK
- U9 pad 59: /CODEC/CODEC_WCLK -> Net-(U9-Pad59)
- U9 pad 61: /CODEC/CODEC_BCLK -> Net-(U9-Pad61)
Routing:
- net /FPGA/X2_L31N: track 42.1 -> 0.00 mm, vias 1 -> 0
- net /FPGA/X2_L31P: track 39.3 -> 0.00 mm, vias 1 -> 0
- net /CODEC/CODEC_BCLK: track 134.7 -> 146.3 mm, vias 1 -> 3
- net /CODEC/CODEC_WCLK: track 136.3 -> 138.8 mm, vias 1 -> 3
- net GND: track 2970.6 -> 2968.3 mm
- net Net-(J_X2-Pad15): track 0.00 -> 0.51 mm
Other:
- board text added: "lboard v2.10.001 2019-12-06"
- board text removed: "lboard v2.9.006 2019-04-06"
